File: h3_extra_ports.kicad_pcb (KiCad board)
At the start: 4 copper layers, 33 x 35.3 mm, 34 parts, among them J1 USB_A, J2 USB_A, J3 USB_A, J4 Conn_02x02_Odd_Even, J5 RS232, J6 Conn_02x12_Odd_Even, J7 Qwiik, J8 Qwiik, J9 Conn_02x12_Odd_Even, U1 MAX3232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

Commit message: Final design - first batch
Parts:
- J5: footprint Connector_IDC:IDC-Header_2x05_P2.54mm_Horizontal -> Connector_PinHeader_2.54mm:PinHeader_2x05_P2.54mm_Horizontal
- moved J5 0.58 mm to (184.8, 66.3)
Connections:
- C11 pad 2: Net-(J2-Pad1) -> (no net)
- C12 pad 2: Net-(J2-Pad1) -> Net-(C11-Pad2)
- C13 pad 2: Net-(J2-Pad1) -> Net-(C11-Pad2)
- C15 pad 2: Net-(J3-Pad1) -> (no net)
- C16 pad 2: Net-(J3-Pad1) -> Net-(C15-Pad2)
- C17 pad 2: Net-(J3-Pad1) -> Net-(C15-Pad2)
- C7 pad 2: Net-(J1-Pad1) -> (no net)
- C8 pad 2: Net-(J1-Pad1) -> Net-(C7-Pad2)
- C9 pad 2: Net-(J1-Pad1) -> Net-(C7-Pad2)
- J1 pad 1: Net-(J1-Pad1) -> Net-(C7-Pad2)
- J2 pad 1: Net-(J2-Pad1) -> Net-(C11-Pad2)
- J3 pad 1: Net-(J3-Pad1) -> Net-(C15-Pad2)
- U2 pad 4: Net-(J1-Pad1) -> Net-(C7-Pad2)
- U3 pad 4: Net-(J2-Pad1) -> Net-(C11-Pad2)
- U4 pad 4: Net-(J3-Pad1) -> Net-(C15-Pad2)
Routing:
- net Net-(J3-Pad1): track 10.5 -> 0.00 mm
- net Net-(C15-Pad2): track 0.00 -> 10.5 mm
- net Net-(J2-Pad1): track 10.5 -> 0.00 mm
- net Net-(C11-Pad2): track 0.00 -> 10.5 mm
- net Net-(J1-Pad1): track 10.5 -> 0.00 mm
- net Net-(C7-Pad2): track 0.00 -> 10.5 mm
