File: h3_extra_ports.kicad_sch (KiCad schematic)
At the start: 34 parts, among them J1 USB_A, J2 USB_A, J3 USB_A, J4 Conn_02x02_Odd_Even, J5 RS232, J6 Conn_02x12_Odd_Even, J7 Qwiik, J8 Qwiik, J9 Conn_02x12_Odd_Even, U1 MAX3232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

Commit message: Final design - first batch
Parts:
- J5: footprint Connector_IDC:IDC-Header_2x05_P2.54mm_Horizontal -> Connector_PinHeader_2.54mm:PinHeader_2x05_P2.54mm_Horizontal
Changed lines of the file:
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@@
     (property "Reference" "J5" (id 0) (at 261.62 141.0802 0))
     (property "Value" "RS232" (id 1) (at 261.62 143.6171 0))
-    (property "Footprint" "Connector_IDC:IDC-Header_2x05_P2.54mm_Horizontal" (id 2) (at 260.35 151.13 0)
+    (property "Footprint" "Connector_PinHeader_2.54mm:PinHeader_2x05_P2.54mm_Horizontal" (id 2) (at 260.35 151.13 0)
       (effects (font (size 1.27 1.27)) hide)
     )
@@
     )
     (path "/a663b413-fda3-44c2-adc3-c85e5335f603"
-      (reference "J5") (unit 1) (value "RS232") (footprint "Connector_IDC:IDC-Header_2x05_P2.54mm_Horizontal")
+      (reference "J5") (unit 1) (value "RS232") (footprint "Connector_PinHeader_2.54mm:PinHeader_2x05_P2.54mm_Horizontal")
     )
     (path "/90c20e3e-0344-4811-8b2b-2d42de31f66d"
